Commit message: Add gazebo support to urdf model

File: src/learning_description/urdf/arm_body.urdf.xacro (robot description, xacro)
@@ -18,5 +18,5 @@
           parent="motor_S"
           xyz="${motor_radius + motor_height/2} 0 0"
-          rpy="0 1.5857963 0"
+          rpy="0 ${pi/2} 0"
   />
   <pole
@@ -25,5 +25,5 @@
           length="${pole_length}"
           xyz="0 ${motor_radius + pole_length/2} 0"
-          rpy="1.5857963 0 0"
+          rpy="${pi/2} 0 0"
   />
   <motor
@@ -31,5 +31,5 @@
           parent="pole_1"
           xyz="0 0 -${pole_length/2 + motor_radius}"
-          rpy="-1.5857963 0 0"
+          rpy="-${pi/2} 0 0"
   />
   <motor
@@ -37,5 +37,5 @@
           parent="motor_U"
           xyz="0 0 ${motor_height/2 + motor_radius}"
-          rpy="-1.5857963 0 0"
+          rpy="-${pi/2} 0 0"
   />
   <pole
@@ -50,5 +50,5 @@
           parent="pole_2"
           xyz="0 0 ${pole_length/2 + motor_radius}"
-          rpy="1.5857963 0 0"
+          rpy="${pi/2} 0 0"
   />
   <motor
@@ -56,5 +56,5 @@
           parent="motor_B"
           xyz="0 0 ${motor_height/2 + motor_radius}"
-          rpy="-1.5857963 0 0"
+          rpy="-${pi/2} 0 0"
   />
   <link name="wrist_link"/>

File: src/learning_description/urdf/arm_parts.urdf.xacro (robot description, xacro)
@@ -1,12 +1,25 @@
 <robot name="arm_body" xmlns:xacro="http://www.ros.org/wiki/xacro">
+  <xacro:property name="pi" value="3.14159265"/>
   <xacro:property name="base_radius" value="0.1"/>
   <xacro:property name="base_height" value="0.01"/>
+  <xacro:property name="base_mass" value="10"/>
   <xacro:property name="motor_radius" value="0.01"/>
   <xacro:property name="motor_height" value="0.02"/>
+  <xacro:property name="motor_mass" value="0.1"/>
   <xacro:property name="pole_radius" value="0.01"/>
   <xacro:property name="pole_length" value="0.2"/>
+  <xacro:property name="pole_mass" value="0.2"/>
   <xacro:property name="standoff_x" value="0"/>
   <xacro:property name="standoff_y" value="0"/>
   <xacro:property name="standoff_z" value="0"/>
+  <xacro:macro name="cylinder_inertial" params="radius length mass">
+    <inertial>
+      <origin xyz="0 0 0" rpy="0 0 0"/>
+      <mass value="${mass}" />
+      <inertia ixx="${0.0833333 * mass * (3 * radius * radius + length * length)}" ixy="0.0" ixz="0.0"
+               iyy="${0.0833333 * mass * (3 * radius * radius + length * length)}" iyz="0.0"
+               izz="${0.5 * mass * radius * radius}" />
+    </inertial>
+  </xacro:macro>
   <xacro:macro name="continuous" params="parent child xyz rpy axis">
     <joint name="${parent}_${child}_joint" type="continuous">
@@ -16,4 +29,12 @@
       <axis xyz="${axis}"/>
     </joint>
+    <transmission name="${parent}_${child}_joint_trans">
+      <type>transmission_interface/SimpleTransmission</type>
+      <joint name="${parent}_${child}_joint"/>
+      <actuator name="${parent}_${child}_joint_motor">
+        <hardwareInterface>VelocityJointInterface</hardwareInterface>
+        <mechanicalReduction>1</mechanicalReduction>
+      </actuator>
+    </transmission>
   </xacro:macro>
   <xacro:macro name="fixed" params="parent child xyz rpy">
@@ -35,4 +56,14 @@
         </material>
       </visual>
+      <collision>
+        <geometry>
+          <cylinder length="${base_height}" radius="${base_radius}"/>
+        </geometry>
+      </collision>
+      <cylinder_inertial
+              radius="${base_radius}"
+              length="${base_height}"
+              mass="${base_mass}"
+      />
     </link>
     <fixed
@@ -42,4 +73,7 @@
             rpy="${rpy}"
     />
+    <gazebo reference="${name}">
+      <material>Gazebo/Yellow</material>
+    </gazebo>
   </xacro:macro>
   <xacro:macro name="motor" params="name parent xyz rpy">
@@ -54,4 +88,14 @@
         </material>
       </visual>
+      <collision>
+        <geometry>
+          <cylinder length="${motor_height}" radius="${motor_radius}"/>
+        </geometry>
+      </collision>
+      <cylinder_inertial
+              radius="${motor_radius}"
+              length="${motor_height}"
+              mass="${motor_mass}"
+      />
     </link>
     <continuous
@@ -62,4 +106,7 @@
             axis="0 0 1"
     />
+    <gazebo reference="${name}">
+      <material>Gazebo/Gray</material>
+    </gazebo>
   </xacro:macro>
   <xacro:macro name="pole" params="name parent length xyz rpy">
@@ -74,4 +121,14 @@
         </material>
       </visual>
+      <collision>
+        <geometry>
+          <cylinder length="${length}" radius="${pole_radius}"/>
+        </geometry>
+      </collision>
+      <cylinder_inertial
+              radius="${pole_radius}"
+              length="${pole_length}"
+              mass="${pole_mass}"
+      />
     </link>
     <fixed
@@ -81,4 +138,7 @@
             rpy="${rpy}"
     />
+    <gazebo reference="${name}">
+      <material>Gazebo/White</material>
+    </gazebo>
   </xacro:macro>
 </robot>

Commit message: Try gazebo_ros_control

File: src/learning_description/urdf/arm_body.urdf.xacro (robot description, xacro)
@@ -11,5 +11,5 @@
           name="motor_S"
           parent="base"
-          xyz="0 0 ${base_height/2 + motor_height/2}"
+          xyz="0 0 ${base_height/2 + motor_height/2 + gap}"
           rpy="0 0 0"
   />
@@ -17,5 +17,5 @@
           name="motor_L"
           parent="motor_S"
-          xyz="${motor_radius + motor_height/2} 0 0"
+          xyz="${motor_radius + motor_height/2 + gap} 0 0"
           rpy="0 ${pi/2} 0"
   />
@@ -24,5 +24,5 @@
           parent="motor_L"
           length="${pole_length}"
-          xyz="0 ${motor_radius + pole_length/2} 0"
+          xyz="0 ${motor_radius + pole_length/2 + gap} 0"
           rpy="${pi/2} 0 0"
   />
@@ -30,5 +30,5 @@
           name="motor_U"
           parent="pole_1"
-          xyz="0 0 -${pole_length/2 + motor_radius}"
+          xyz="0 0 -${pole_length/2 + motor_radius + gap}"
           rpy="-${pi/2} 0 0"
   />
@@ -36,5 +36,5 @@
           name="motor_R"
           parent="motor_U"
-          xyz="0 0 ${motor_height/2 + motor_radius}"
+          xyz="0 0 ${motor_height/2 + motor_radius + gap}"
           rpy="-${pi/2} 0 0"
   />
@@ -43,5 +43,5 @@
           parent="motor_R"
           length="${pole_length}"
-          xyz="0 0 ${motor_height/2 + pole_length/2}"
+          xyz="0 0 ${motor_height/2 + pole_length/2 + gap}"
           rpy="0 0 0"
   />
@@ -49,5 +49,5 @@
           name="motor_B"
           parent="pole_2"
-          xyz="0 0 ${pole_length/2 + motor_radius}"
+          xyz="0 0 ${pole_length/2 + motor_radius + gap}"
           rpy="${pi/2} 0 0"
   />
@@ -55,5 +55,5 @@
           name="motor_T"
           parent="motor_B"
-          xyz="0 0 ${motor_height/2 + motor_radius}"
+          xyz="0 0 ${motor_height/2 + motor_radius + gap}"
           rpy="-${pi/2} 0 0"
   />
@@ -62,5 +62,5 @@
           parent="motor_T"
           child="wrist_link"
-          xyz="0 0 ${motor_height/2}"
+          xyz="0 0 ${motor_height/2 + gap}"
           rpy="0 0 0"
   />

File: src/learning_description/urdf/arm_parts.urdf.xacro (robot description, xacro)
@@ -1,4 +1,5 @@
 <robot name="arm_body" xmlns:xacro="http://www.ros.org/wiki/xacro">
   <xacro:property name="pi" value="3.14159265"/>
+  <xacro:property name="gap" value="0.001"/>
   <xacro:property name="base_radius" value="0.1"/>
   <xacro:property name="base_height" value="0.01"/>
@@ -6,11 +7,17 @@
   <xacro:property name="motor_radius" value="0.01"/>
   <xacro:property name="motor_height" value="0.02"/>
-  <xacro:property name="motor_mass" value="0.1"/>
+  <xacro:property name="motor_mass" value="1"/>
   <xacro:property name="pole_radius" value="0.01"/>
   <xacro:property name="pole_length" value="0.2"/>
-  <xacro:property name="pole_mass" value="0.2"/>
+  <xacro:property name="pole_mass" value="2"/>
   <xacro:property name="standoff_x" value="0"/>
   <xacro:property name="standoff_y" value="0"/>
   <xacro:property name="standoff_z" value="0"/>
+  <gazebo>
+    <plugin filename="libgazebo_ros_control.so" name="ros_control">
+      <robotNamespace>/</robotNamespace>
+      <legacyModeNS>true</legacyModeNS>
+    </plugin>
+  </gazebo>
   <xacro:macro name="cylinder_inertial" params="radius length mass">
     <inertial>
@@ -31,7 +38,9 @@
     <transmission name="${parent}_${child}_joint_trans">
       <type>transmission_interface/SimpleTransmission</type>
-      <joint name="${parent}_${child}_joint"/>
+      <joint name="${parent}_${child}_joint">
+        <hardwareInterface>hardware_interface/PositionJointInterface</hardwareInterface>
+      </joint>
       <actuator name="${parent}_${child}_joint_motor">
-        <hardwareInterface>VelocityJointInterface</hardwareInterface>
+        <hardwareInterface>hardware_interface/PositionJointInterface</hardwareInterface>
         <mechanicalReduction>1</mechanicalReduction>
       </actuator>

Commit message: Add gazebo_ros_control support to urdf model

File: src/learning_description/urdf/arm_body.urdf.xacro (robot description, xacro)
@@ -1,67 +1,77 @@
 <robot name="arm_body" xmlns:xacro="http://www.ros.org/wiki/xacro">
   <xacro:include filename="$(find learning_description)/urdf/arm_parts.urdf.xacro"/>
-  <link name="base_link"/>
-  <base
-          name="base"
-          parent="base_link"
-          xyz="${standoff_x} ${standoff_y} ${standoff_z + base_height/2}"
-          rpy="0 0 0"
-  />
-  <motor
-          name="motor_S"
-          parent="base"
-          xyz="0 0 ${base_height/2 + motor_height/2 + gap}"
-          rpy="0 0 0"
-  />
-  <motor
-          name="motor_L"
-          parent="motor_S"
-          xyz="${motor_radius + motor_height/2 + gap} 0 0"
-          rpy="0 ${pi/2} 0"
-  />
-  <pole
-          name="pole_1"
-          parent="motor_L"
-          length="${pole_length}"
-          xyz="0 ${motor_radius + pole_length/2 + gap} 0"
-          rpy="${pi/2} 0 0"
-  />
-  <motor
-          name="motor_U"
-          parent="pole_1"
-          xyz="0 0 -${pole_length/2 + motor_radius + gap}"
-          rpy="-${pi/2} 0 0"
-  />
-  <motor
-          name="motor_R"
-          parent="motor_U"
-          xyz="0 0 ${motor_height/2 + motor_radius + gap}"
-          rpy="-${pi/2} 0 0"
-  />
-  <pole
-          name="pole_2"
-          parent="motor_R"
-          length="${pole_length}"
-          xyz="0 0 ${motor_height/2 + pole_length/2 + gap}"
-          rpy="0 0 0"
-  />
-  <motor
-          name="motor_B"
-          parent="pole_2"
-          xyz="0 0 ${pole_length/2 + motor_radius + gap}"
-          rpy="${pi/2} 0 0"
-  />
-  <motor
-          name="motor_T"
-          parent="motor_B"
-          xyz="0 0 ${motor_height/2 + motor_radius + gap}"
-          rpy="-${pi/2} 0 0"
-  />
-  <link name="wrist_link"/>
-  <fixed
-          parent="motor_T"
-          child="wrist_link"
-          xyz="0 0 ${motor_height/2 + gap}"
-          rpy="0 0 0"
-  />
+  <xacro:macro name="arm_body">
+    <plugin_ros_control/>
+    <plugin_joint_state_publisher>
+      <jointName>
+        motor_S_joint, motor_L_joint, motor_U_joint,
+        motor_R_joint, motor_B_joint, motor_T_joint
+      </jointName>
+    </plugin_joint_state_publisher>
+    <link name="base_link"/>
+    <base
+            name="base"
+            parent="base_link"
+            xyz="${standoff_x} ${standoff_y} ${standoff_z + base_height/2 + gap}"
+            rpy="0 0 0"
+    />
+    <motor
+            name="motor_S"
+            parent="base"
+            xyz="0 0 ${base_height/2 + motor_height/2 + gap}"
+            rpy="0 0 0"
+    />
+    <motor
+            name="motor_L"
+            parent="motor_S"
+            xyz="${motor_radius + motor_height/2 + gap} 0 0"
+            rpy="0 ${pi/2} 0"
+    />
+    <pole
+            name="pole_1"
+            parent="motor_L"
+            length="${pole_length}"
+            xyz="0 ${motor_radius + pole_length/2 + gap} 0"
+            rpy="${pi/2} 0 0"
+    />
+    <motor
+            name="motor_U"
+            parent="pole_1"
+            xyz="0 0 -${pole_length/2 + motor_radius + gap}"
+            rpy="-${pi/2} 0 0"
+    />
+    <motor
+            name="motor_R"
+            parent="motor_U"
+            xyz="0 0 ${motor_height/2 + motor_radius + gap}"
+            rpy="-${pi/2} 0 0"
+    />
+    <pole
+            name="pole_2"
+            parent="motor_R"
+            length="${pole_length}"
+            xyz="0 0 ${motor_height/2 + pole_length/2 + gap}"
+            rpy="0 0 0"
+    />
+    <motor
+            name="motor_B"
+            parent="pole_2"
+            xyz="0 0 ${pole_length/2 + motor_radius + gap}"
+            rpy="${pi/2} 0 0"
+    />
+    <motor
+            name="motor_T"
+            parent="motor_B"
+            xyz="0 0 ${motor_height/2 + motor_radius + gap}"
+            rpy="-${pi/2} 0 0"
+    />
+    <link name="wrist_link"/>
+    <fixed
+            name="wrist_joint"
+            parent="motor_T"
+            child="wrist_link"
+            xyz="0 0 ${motor_height/2 + gap}"
+            rpy="0 0 0"
+    />
+  </xacro:macro>
 </robot>

File: src/learning_description/urdf/arm_description.urdf.xacro (robot description, xacro)
@@ -2,3 +2,9 @@
   <xacro:include filename="$(find learning_description)/urdf/arm_body.urdf.xacro"/>
   <arm_body/>
+  <link name="world"/>
+  <joint name="world_joint" type="fixed">
+    <parent link="world" />
+    <child link = "base_link" />
+    <origin xyz="0.0 0.0 0" rpy="0.0 0.0 0.0" />
+  </joint>
 </robot>

File: src/learning_description/urdf/arm_parts.urdf.xacro (robot description, xacro)
@@ -1,23 +1,39 @@
 <robot name="arm_body" xmlns:xacro="http://www.ros.org/wiki/xacro">
+  <!-- property -->
   <xacro:property name="pi" value="3.14159265"/>
-  <xacro:property name="gap" value="0.001"/>
-  <xacro:property name="base_radius" value="0.1"/>
-  <xacro:property name="base_height" value="0.01"/>
-  <xacro:property name="base_mass" value="10"/>
+  <xacro:property name="gap" value="0.0"/>
+  <xacro:property name="base_radius" value="0.01"/>
+  <xacro:property name="base_height" value="0.02"/>
+  <xacro:property name="base_mass" value="1"/>
   <xacro:property name="motor_radius" value="0.01"/>
   <xacro:property name="motor_height" value="0.02"/>
   <xacro:property name="motor_mass" value="1"/>
+  <xacro:property name="motor_effort" value="150.0"/>
+  <xacro:property name="motor_vel" value="${pi}"/>
   <xacro:property name="pole_radius" value="0.01"/>
-  <xacro:property name="pole_length" value="0.2"/>
-  <xacro:property name="pole_mass" value="2"/>
+  <xacro:property name="pole_length" value="0.1"/>
+  <xacro:property name="pole_mass" value="5"/>
   <xacro:property name="standoff_x" value="0"/>
   <xacro:property name="standoff_y" value="0"/>
   <xacro:property name="standoff_z" value="0"/>
-  <gazebo>
-    <plugin filename="libgazebo_ros_control.so" name="ros_control">
-      <robotNamespace>/</robotNamespace>
-      <legacyModeNS>true</legacyModeNS>
-    </plugin>
-  </gazebo>
+  <!-- plugin -->
+  <xacro:macro name="plugin_ros_control">
+    <gazebo>
+      <plugin filename="libgazebo_ros_control.so" name="ros_control">
+        <robotNamespace>/</robotNamespace>
+        <legacyModeNS>true</legacyModeNS>
+      </plugin>
+    </gazebo>
+  </xacro:macro>
+  <xacro:macro name="plugin_joint_state_publisher" params="*jointName">
+    <gazebo>
+      <plugin filename="libgazebo_ros_joint_state_publisher.so" name="joint_state_publisher">
+        <xacro:insert_block name="jointName"/>
+        <updateRate>50</updateRate>
+        <alwaysOn>true</alwaysOn>
+      </plugin>
+    </gazebo>
+  </xacro:macro>
+  <!-- inertial -->
   <xacro:macro name="cylinder_inertial" params="radius length mass">
     <inertial>
@@ -29,17 +45,20 @@
     </inertial>
   </xacro:macro>
-  <xacro:macro name="continuous" params="parent child xyz rpy axis">
-    <joint name="${parent}_${child}_joint" type="continuous">
+  <!-- joint -->
+  <xacro:macro name="continuous" params="name parent child xyz rpy axis">
+    <joint name="${name}" type="continuous">
       <parent link="${parent}"/>
       <child link="${child}"/>
       <origin xyz="${xyz}" rpy="${rpy}"/>
       <axis xyz="${axis}"/>
+      <limit effort="${motor_effort}" velocity="${motor_vel}"/>
+      <dynamics damping="0.0" friction="0.0"/>
     </joint>
-    <transmission name="${parent}_${child}_joint_trans">
+    <transmission name="${name}_trans">
       <type>transmission_interface/SimpleTransmission</type>
-      <joint name="${parent}_${child}_joint">
+      <joint name="${name}">
         <hardwareInterface>hardware_interface/PositionJointInterface</hardwareInterface>
       </joint>
-      <actuator name="${parent}_${child}_joint_motor">
+      <actuator name="${name}_motor">
         <hardwareInterface>hardware_interface/PositionJointInterface</hardwareInterface>
         <mechanicalReduction>1</mechanicalReduction>
@@ -47,6 +66,6 @@
     </transmission>
   </xacro:macro>
-  <xacro:macro name="fixed" params="parent child xyz rpy">
-    <joint name="${parent}_${child}_joint" type="fixed">
+  <xacro:macro name="fixed" params="name parent child xyz rpy">
+    <joint name="${name}" type="fixed">
       <parent link="${parent}"/>
       <child link="${child}"/>
@@ -54,4 +73,5 @@
     </joint>
   </xacro:macro>
+  <!-- link -->
   <xacro:macro name="base" params="name parent xyz rpy">
     <link name="${name}">
@@ -77,4 +97,5 @@
     </link>
     <fixed
+            name="${name}_joint"
             parent="${parent}"
             child="${name}"
@@ -109,4 +130,5 @@
     </link>
     <continuous
+            name="${name}_joint"
             parent="${parent}"
             child="${name}"
@@ -142,4 +164,5 @@
     </link>
     <fixed
+            name="${name}_joint"
             parent="${parent}"
             child="${name}"

Commit message: Better arm_description package

File: src/learning_description/urdf/arm_body.urdf.xacro (robot description, xacro)
@@ -3,10 +3,4 @@
   <xacro:macro name="arm_body">
     <plugin_ros_control/>
-    <plugin_joint_state_publisher>
-      <jointName>
-        motor_S_joint, motor_L_joint, motor_U_joint,
-        motor_R_joint, motor_B_joint, motor_T_joint
-      </jointName>
-    </plugin_joint_state_publisher>
     <link name="base_link"/>
     <base

File: src/learning_description/urdf/arm_description.urdf.xacro (robot description, xacro)
@@ -1,10 +1,4 @@
 <robot name="arm_robot" xmlns:xacro="http://www.ros.org/wiki/xacro">
   <xacro:include filename="$(find learning_description)/urdf/arm_body.urdf.xacro"/>
-  <arm_body/>
-  <link name="world"/>
-  <joint name="world_joint" type="fixed">
-    <parent link="world" />
-    <child link = "base_link" />
-    <origin xyz="0.0 0.0 0" rpy="0.0 0.0 0.0" />
-  </joint>
+  <xacro:include filename="$(find learning_description)/urdf/arm_hand.urdf.xacro"/>
 </robot>

File: src/learning_description/urdf/arm_parts.urdf.xacro (robot description, xacro)
@@ -3,14 +3,14 @@
   <xacro:property name="pi" value="3.14159265"/>
   <xacro:property name="gap" value="0.0"/>
-  <xacro:property name="base_radius" value="0.01"/>
-  <xacro:property name="base_height" value="0.02"/>
+  <xacro:property name="base_radius" value="0.05"/>
+  <xacro:property name="base_height" value="0.1"/>
   <xacro:property name="base_mass" value="10"/>
-  <xacro:property name="motor_radius" value="0.01"/>
-  <xacro:property name="motor_height" value="0.02"/>
+  <xacro:property name="motor_radius" value="0.05"/>
+  <xacro:property name="motor_height" value="0.1"/>
   <xacro:property name="motor_mass" value="10"/>
   <xacro:property name="motor_effort" value="150.0"/>
   <xacro:property name="motor_vel" value="${pi}"/>
-  <xacro:property name="pole_radius" value="0.01"/>
-  <xacro:property name="pole_length" value="0.1"/>
+  <xacro:property name="pole_radius" value="0.05"/>
+  <xacro:property name="pole_length" value="0.5"/>
   <xacro:property name="pole_mass" value="50"/>
   <xacro:property name="standoff_x" value="0"/>
@@ -23,13 +23,4 @@
         <robotNamespace>/</robotNamespace>
         <legacyModeNS>true</legacyModeNS>
-      </plugin>
-    </gazebo>
-  </xacro:macro>
-  <xacro:macro name="plugin_joint_state_publisher" params="*jointName">
-    <gazebo>
-      <plugin filename="libgazebo_ros_joint_state_publisher.so" name="joint_state_publisher">
-        <xacro:insert_block name="jointName"/>
-        <updateRate>50</updateRate>
-        <alwaysOn>true</alwaysOn>
       </plugin>
     </gazebo>

File: src/learning_moveit/urdf/robot.urdf.xacro (robot description, xacro)
@@ -1,4 +1,5 @@
 <?xml version="1.0" ?>
 <robot name="arm_robot" xmlns:xacro="http://www.ros.org/wiki/xacro">
+    <!-- arm -->
     <xacro:include filename="$(find learning_description)/urdf/arm_body.urdf.xacro"/>
     <arm_body/>
