Commit message: Add arm_common.py

File: src/arm_common/urdf/arm_common.urdf.xacro (robot description, xacro)
@@ -105,5 +105,5 @@
           <cylinder length="${motor_height}" radius="${motor_radius}"/>
         </geometry>
-        <material name="gray">
+        <material name="grey">
           <color rgba="0.75 0.75 0.75 1"/>
         </material>
@@ -129,5 +129,5 @@
     />
     <gazebo reference="${name}">
-      <material>Gazebo/Gray</material>
+      <material>Gazebo/Grey</material>
     </gazebo>
   </xacro:macro>

Commit message: Better arm model

File: src/arm_common/urdf/arm_common.urdf.xacro (robot description, xacro)
@@ -150,6 +150,6 @@
       <cylinder_inertial
               radius="${pole_radius}"
-              length="${pole_length}"
-              mass="${pole_mass}"
+              length="${length}"
+              mass="${pole_mass*(length/pole_length)}"
       />
     </link>

File: src/arm_description/urdf/arm_description.urdf.xacro (robot description, xacro)
@@ -3,5 +3,7 @@
   <xacro:macro name="arm">
     <plugin_ros_control/>
+    <!--    base_link    -->
     <link name="base_link"/>
+    <!--    shoulder    -->
     <base
             name="base"
@@ -11,18 +13,19 @@
     />
     <motor
-            name="motor_S"
+            name="shoulder_pan"
             parent="base"
             xyz="0 0 ${base_height/2 + motor_height/2 + gap}"
             rpy="0 0 0"
     />
+    <!--    upper arm    -->
     <motor
-            name="motor_L"
-            parent="motor_S"
+            name="shoulder_lift"
+            parent="shoulder_pan"
             xyz="${motor_radius + motor_height/2 + gap} 0 0"
             rpy="0 ${pi/2} 0"
     />
     <pole
-            name="pole_1"
-            parent="motor_L"
+            name="upper_arm"
+            parent="shoulder_lift"
             length="${pole_length}"
             xyz="0 ${motor_radius + pole_length/2 + gap} 0"
@@ -30,38 +33,48 @@
     />
     <motor
-            name="motor_U"
-            parent="pole_1"
+            name="elbow"
+            parent="upper_arm"
             xyz="0 0 -${pole_length/2 + motor_radius + gap}"
             rpy="-${pi/2} 0 0"
     />
-    <motor
-            name="motor_R"
-            parent="motor_U"
+    <!--    fore arm    -->
+    <pole
+            name="fore_arm_elbow"
+            parent="elbow"
+            length="${motor_height}"
             xyz="0 0 ${motor_height/2 + motor_radius + gap}"
             rpy="-${pi/2} 0 0"
     />
     <pole
-            name="pole_2"
-            parent="motor_R"
+            name="fore_arm"
+            parent="fore_arm_elbow"
             length="${pole_length}"
-            xyz="0 0 ${motor_height/2 + pole_length/2 + gap}"
+            xyz="0 0 ${pole_length/2 + motor_height/2 + gap}"
             rpy="0 0 0"
     />
+    <!--    wrist    -->
     <motor
-            name="motor_B"
-            parent="pole_2"
+            name="wrist_1"
+            parent="fore_arm"
             xyz="0 0 ${pole_length/2 + motor_radius + gap}"
             rpy="${pi/2} 0 0"
     />
     <motor
-            name="motor_T"
-            parent="motor_B"
+            name="wrist_2"
+            parent="wrist_1"
             xyz="0 0 ${motor_height/2 + motor_radius + gap}"
             rpy="-${pi/2} 0 0"
     />
+    <motor
+            name="wrist_3"
+            parent="wrist_2"
+            xyz="0 0 ${motor_height/2 + motor_radius + gap}"
+            rpy="${pi/2} 0 0"
+    />
+    <!--    wrist_link    -->
     <link name="wrist_link"/>
     <fixed
             name="wrist_joint"
-            parent="motor_T"
+            parent="wrist_3"
             child="wrist_link"
             xyz="0 0 ${motor_height/2 + gap}"

File: src/arm_shand_description/urdf/arm_shand_description.urdf.xacro (robot description, xacro)
@@ -1,9 +1,11 @@
 <robot name="arm_shand" xmlns:xacro="http://www.ros.org/wiki/xacro">
-  <xacro:property name="finger_x" value="0.05"/>
+  <xacro:property name="wrist_length" value="0.02"/>
+  <xacro:property name="palm_thick" value="0.02"/>
+  <xacro:property name="finger_x" value="0.08"/>
   <xacro:property name="finger_y" value="0.02"/>
   <xacro:property name="finger_length" value="0.1"/>
   <xacro:property name="finger_lower" value="${finger_y/2}"/>
-  <xacro:property name="finger_upper" value="${finger_y/2 + 0.06}"/>
-  <xacro:property name="finger_mass" value="1"/>
+  <xacro:property name="finger_upper" value="${finger_y/2 + 0.08}"/>
+  <xacro:property name="finger_mass" value="5"/>
   <xacro:include filename="$(find arm_description)/urdf/arm_description.urdf.xacro"/>
   <xacro:macro name="prismatic" params="name parent child xyz rpy axis lower upper">
@@ -63,21 +65,67 @@
     </gazebo>
   </xacro:macro>
+  <xacro:macro name="palm" params="name parent xyz rpy">
+    <link name="${name}">
+      <visual>
+        <origin xyz="0 0 0" rpy="0 0 0"/>
+        <geometry>
+          <box size="${finger_x} ${finger_upper*2} ${palm_thick}"/>
+        </geometry>
+        <material name="white">
+          <color rgba="1 1 1 1"/>
+        </material>
+      </visual>
+      <collision>
+        <geometry>
+          <box size="${finger_x} ${finger_upper*2} ${palm_thick}"/>
+        </geometry>
+      </collision>
+      <cylinder_inertial
+              radius="${finger_x/4+(finger_upper*2)/4}"
+              length="${palm_thick}"
+              mass="${finger_mass}"
+      />
+    </link>
+    <fixed
+            name="${name}_joint"
+            parent="${parent}"
+            child="${name}"
+            xyz="${xyz}"
+            rpy="${rpy}"
+    />
+    <gazebo reference="${name}">
+      <material>Gazebo/White</material>
+    </gazebo>
+  </xacro:macro>
   <!-- simple hand -->
   <xacro:macro name="arm_shand">
     <arm/>
+    <pole
+            name="sh_wrist"
+            parent="wrist_link"
+            length="${wrist_length}"
+            xyz="0 0 ${wrist_length/2}"
+            rpy="0 0 0"
+    />
+    <palm
+            name="sh_palm"
+            parent="sh_wrist"
+            xyz="0 0 ${wrist_length/2 + palm_thick/2}"
+            rpy="0 0 0"
+    />
     <!-- end effector -->
     <finger
-            name="finger1"
-            parent="motor_T"
+            name="sh_finger1"
+            parent="sh_palm"
             length="${finger_length}"
-            xyz="0 0 ${motor_height/2 + gap + finger_length/2}"
-            rpy="0 0 0"
+            xyz="0 0 ${palm_thick/2 + gap + finger_length/2}"
+            rpy="0 0 3.1415926"
     />
     <finger
-            name="finger2"
-            parent="motor_T"
+            name="sh_finger2"
+            parent="sh_palm"
             length="${finger_length}"
-            xyz="0 0 ${motor_height/2 + gap + finger_length/2}"
-            rpy="0 0 3.1415926"
+            xyz="0 0 ${palm_thick/2 + gap + finger_length/2}"
+            rpy="0 0 0"
     />
   </xacro:macro>
