Commit message: Optimize place method of arm

File: src/arm_shand_description/urdf/arm_shand_description.urdf.xacro (robot description, xacro)
@@ -8,4 +8,6 @@
   <xacro:property name="finger_upper" value="${finger_y/2 + 0.08}"/>
   <xacro:property name="finger_mass" value="5"/>
+  <xacro:property name="finger_effort" value="500.0"/>
+  <xacro:property name="finger_vel" value="${pi}"/>
   <xacro:include filename="$(find arm_description)/urdf/arm_description.urdf.xacro"/>
   <xacro:macro name="prismatic" params="name parent child xyz rpy axis lower upper">
@@ -15,6 +17,6 @@
       <origin xyz="${xyz}" rpy="${rpy}"/>
       <axis xyz="${axis}"/>
-      <limit effort="${motor_effort}" velocity="${motor_vel}" lower="${lower}" upper="${upper}"/>
-      <dynamics damping="0.0" friction="1"/>
+      <limit effort="${finger_effort}" velocity="${finger_vel}" lower="${lower}" upper="${upper}"/>
+      <dynamics damping="0.0" friction="0.0"/>
     </joint>
     <transmission name="${name}_trans">
